File: design/source/kicad/P-1000072_Cicada Wi-Fi.sch (KiCad schematic (older format))
At the start: 66 parts, among them J3 Host, U1 HX3406, U3 ESP-07S

Commit message: WiFi Cicada First Design and Manufacturing files release
Parts:
- J3: footprint edemame-custom-footprints:PinSocket_2x08_P2.54mm_Vertical_padded -> Cicada-footprints:PinSocket_2x08_P2.54mm_Vertical_padded
- L2: footprint edemame-custom-footprints:L_4030_Handsoldering -> Cicada-footprints:L_4030_Handsoldering
- LOGO1: footprint edemame-custom-footprints:okra_logo_copper_2 -> Cicada-footprints:okra_logo_copper_2
- TP1, TP12, TP13, TP14, TP15, TP16, TP3: footprint edemame-custom-footprints:TestPoint_Pad_D1.5mm -> okra-footprints:TestPoint_Pad_D1.5mm
- TP23, TP24, TP25, TP26, TP27, TP28, TP29, TP30, TP32, TP33, TP34, TP35, TP4, TP5, TP6, TP7, TP8, TP9: footprint edemame-custom-footprints:TestPoint_Pad_D1.5mm -> okra-footprints:TestPoint_Pad_D1.5mm; symbol ATE-ACQ-rescue:TestPoint-Connector -> Connector:TestPoint
- U3: footprint edemame-custom-footprints:ESP-07S -> Cicada-footprints:ESP-07S

Commit message: deleted previous production files, reviewed SCH and PCB files
Parts:
- added TP10: GND, okra-footprints:TestPoint_Pad_D1.5mm, symbol Connector:TestPoint
- R13: value 22.6K -> 340k; MPN 0402WGF2262TCE -> 0402WGF5492TCE; SRCPN C26960 -> (none)
Connections:
- net 3V3: no longer R12.1, R13.1
- net GND: now also TP10.1
- net Vref(3V3): now also R12.1, R13.1
Other:
- note added: "VER_2 = 3"
- note removed: "Icc-B (Pout=26dbm, 11Mbps cck sigal, BT =0.45 = 560mA"
- note removed: "Icc-G (Pout=23dBm, 54Mbps OFdm signal, 64QAM) = 460mA"
- note removed: "Icc_OFF (EN=0V, No RF Applied) = 100uA"
- note removed: "SE2604L"
- note removed: "VER_2 = 0"
- moved on the sheet: C1, C14, C16, C19, C2, C20, C21, C22, C24, C29, C3, C4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

Commit message: 1.Schematics improvement and crediblity (cleared empty spaces, improved read me and reviewed and cleaned component spec mismatch 2.PCB improments (cleaned top layer copper zones, cleaned vias and updated production release verion on the pcb silk screen 3.BOM mismatch (R13 changed to output board version number 6.3, previously R13 was DNP)
Parts:
- added TP39: GND, okra-footprints:TestPoint_Pad_D1.5mm, symbol P-1000072_Cicada-Wi-Fi-rescue:TestPoint-Connector-P-1000072_Cicada-Wi-Fi-rescue
- C1, C2, C21, C22, C24: symbol Device:CP_Small -> P-1000072_Cicada-Wi-Fi-rescue:CP_Small-Device-P-1000072_Cicada-Wi-Fi-rescue
- C14, C16, C19, C20, C29, C3, C4, C6, C8, C9: symbol Device:C_Small -> P-1000072_Cicada-Wi-Fi-rescue:C_Small-Device-P-1000072_Cicada-Wi-Fi-rescue
- FID1, FID2, FID3, FID4, FID5, FID6: symbol Mechanical:Fiducial -> P-1000072_Cicada-Wi-Fi-rescue:Fiducial-Mechanical-P-1000072_Cicada-Wi-Fi-rescue
- H1, H2: symbol Mechanical:MountingHole_Pad -> P-1000072_Cicada-Wi-Fi-rescue:MountingHole_Pad-Mechanical-P-1000072_Cicada-Wi-Fi-rescue
- J3: symbol connector:Conn_02x8_Odd_Even_Side_padding -> P-1000072_Cicada-Wi-Fi-rescue:Conn_02x8_Odd_Even_Side_padding-connector-P-1000072_Cicada-Wi-Fi-rescue
- L2: symbol Device:L_Small -> P-1000072_Cicada-Wi-Fi-rescue:L_Small-Device-P-1000072_Cicada-Wi-Fi-rescue
- LOGO1: symbol Graphic:SYM_Hot_Small -> P-1000072_Cicada-Wi-Fi-rescue:SYM_Hot_Small-Graphic-P-1000072_Cicada-Wi-Fi-rescue
- PCB1: symbol Okra_misc:PCB -> P-1000072_Cicada-Wi-Fi-rescue:PCB-Okra_misc-P-1000072_Cicada-Wi-Fi-rescue
- R1, R10, R11, R12, R4, R5, R6, R7, R8, R9: symbol Device:R_Small -> P-1000072_Cicada-Wi-Fi-rescue:R_Small-Device-P-1000072_Cicada-Wi-Fi-rescue
- R13: value 340k -> 86.6k; symbol Device:R_Small -> P-1000072_Cicada-Wi-Fi-rescue:R_Small-Device-P-1000072_Cicada-Wi-Fi-rescue; DNP DNP -> (none); MPN 0402WGF5492TCE -> 0402WGF8662TCE; SRCPN (none) -> C423187
- TP1, TP10, TP12, TP13, TP14, TP15, TP16, TP2, TP23, TP24, TP25, TP26, TP27, TP28, TP29, TP3, TP30, TP32, TP33, TP34, TP35, TP4, TP5, TP6, TP7, TP8, TP9: symbol Connector:TestPoint -> P-1000072_Cicada-Wi-Fi-rescue:TestPoint-Connector-P-1000072_Cicada-Wi-Fi-rescue
- U1: symbol Regulator_Switching:LTC3406ES5 -> P-1000072_Cicada-Wi-Fi-rescue:LTC3406ES5-Regulator_Switching-P-1000072_Cicada-Wi-Fi-rescue
- U3: symbol RF_Module:ESP-07S -> P-1000072_Cicada-Wi-Fi-rescue:ESP-07S-RF_Module-P-1000072_Cicada-Wi-Fi-rescue
Connections:
- net GND: now also TP39.1
Other:
- note added: "Fiducials, Munting Holes, Logos, PCB"
- note added: "HOST CONNECTOR"
- note added: "Power Consumption:"
- note added: "Power Supply HX3406 max output:"
- note added: "The two pins Ver_1 and Ver_2 allow the host board/MCU to detect \nwhat type and version of communication board is connected.\nEach Ver_1/2 pin has a 40.2k resistor to GND on the host side, and \nthe resisitor loaded on the Cicada dagughter board (this PCB) \ncreates a voltage divider that is then read by the host MCU as an \nanalog voltage\n\nThe Ver_1 pin describes the type of Cicada comms board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"
- note added: "VER_1\n(Cicada type)"
- note added: "WIFI Module ESP-07S Consumption:"
- note added: "We use a 2x10 female pin socket as it fits perfectly in a 2x8\nshrouded pin header on the host side. We don't use a 2x8 \npin socket as it is narrower than a 2x8 shrouded header \nand can allowing off-by-1 pin insertion. We don't use a 2x8 \nkeyed pin sockets are they seem to be very uncommon."
- note removed: "ESP-07S"
- note removed: "Electrical char:"
- note removed: "HX3406"
- note removed: "Host connector"
- note removed: "Maj version"
- note removed: "The version resistor forms a voltage divider with a\n40.2K resistor on the host board. The host then can\nread the version as an analog voltage value.\nCheck out the table."
- note removed: "We use a 2x10 female pin socket that fits perfectly in a 2x8\nshrouded pin header on the host side. A 2x8 shrouded header\nis wider than a 2x8 socket, allowing off-by-1 pin insertion.\n\nKeyed female sockets are very uncommon."
- moved on the sheet: C1, C14, C16, C19, C2, C20, C21, C22, C24, C29, C3, C4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
